Commit message: unfinished leapmotion
unfinished leapmotion
wait leap arrive to test

File: Hard/ProjectAliceMK1/robots/ProjectAliceMK1.URDF (robot description, URDF)
Before this commit: robot ProjectAliceMK1, 14 links, 13 joints
Joints:
- joint L1L: limit lower=-1.7 upper=1.7 effort=10 velocity=1 -> lower=-1.7 upper=0 effort=10 velocity=1
- joint R1R: limit lower=-1.7 upper=1.7 effort=10 velocity=1 -> lower=0 upper=1.7 effort=10 velocity=1
